File: pcb/ver0.2/main_rigid_board_kicad_project/msa.kicad_pcb (KiCad board)
At the start: 2 copper layers, 47.8 x 9.4 mm, 50 parts, among them J1 USB_B_Micro, J2 SWD Prog, U1 MCP1702, U2 MCP73831-2-OT, U3 W25Q128JV, U4 RP2040, U5 ‎DMP21D0UT-7‎, Y1 H130B-12.000-20-3050-EXT-TR

Commit message: latest working mic array
Parts:
- added H1: MountingHole, OpenSourceSmartGlasses:Mount_hole_small_0.7mm, F.Cu at (162.7, 90.1)
- added H2: MountingHole, OpenSourceSmartGlasses:Mount_hole_small_0.7mm, F.Cu at (122.1, 86.5)
- added SW1: SW_SPST, Button_Switch_SMD:SW_SPST_B3U-3100P-B, B.Cu at (151.2, 83.7)
- CONN1: footprint OpenSourceSmartGlasses:slim_stack_molex_PLUG_5035521222 -> OpenSourceSmartGlasses:slim_stack_molex_RECEPTACLE_5035481222
- D1: moved to F.Cu
- D2: footprint Capacitor_SMD:C_0402_1005Metric_Pad0.74x0.62mm_HandSolder -> LED_SMD:LED_0402_1005Metric
- R6: moved to B.Cu
- moved R4 15.4 mm to (141.0, 87.3)
- moved R5 15.4 mm to (141.0, 88.3)
- moved BT1 13.1 mm to (162.6, 87.9), turned to 90 degrees
- moved TP4 5.89 mm to (154.9, 87.0)
- moved TP1 3.53 mm to (146.6, 85.3), turned to -90 degrees
- moved D1 1.80 mm to (139.2, 82.7)
- moved R6 1.20 mm to (137.9, 82.6)
- moved CONN1 0.69 mm to (118.5, 88.8)
- moved C1 0.45 mm to (162.3, 87.6)
- moved C5 0.45 mm to (157.4, 89.0)
- moved U1 0.45 mm to (159.9, 88.7)
- moved TP9 0.30 mm to (121.2, 83.8)
- moved C19 0.20 mm to (122.4, 83.7)
Connections:
- CONN1 pad 1: unconnected-(CONN1-Pad1) -> +3V3
- CONN1 pad 10: /MIC_DOUT_3 -> /MIC_DOUT_2
- CONN1 pad 11: -BATT -> /MIC_DOUT_1
- CONN1 pad 12: unconnected-(CONN1-Pad12) -> /MIC_DOUT_0
- CONN1 pad 2: unconnected-(CONN1-Pad2) -> /MIC_CLK
- CONN1 pad 5: /MIC_CLK -> unconnected-(CONN1-Pad5)
- CONN1 pad 6: +3V3 -> unconnected-(CONN1-Pad6)
- CONN1 pad 7: /MIC_DOUT_0 -> unconnected-(CONN1-Pad7)
- CONN1 pad 8: /MIC_DOUT_1 -> -BATT
- CONN1 pad 9: /MIC_DOUT_2 -> /MIC_DOUT_3
- D1 pad 1: -BATT -> Net-(D1-Pad1)
- D1 pad 2: Net-(D1-Pad2) -> /RED_LED
- R6 pad 1: Net-(D1-Pad2) -> -BATT
- R6 pad 2: /RED_LED -> Net-(D1-Pad1)
Routing:
- net /USB-D_P: track 20.3 -> 2.78 mm
- net /USB0-D_P: track 3.39 -> 20.9 mm
- net /USB0-D_N: track 4.24 -> 21.7 mm
- net /USB-D_N: track 20.1 -> 2.94 mm
- net +BATT: track 10.8 -> 23.3 mm, vias 1 -> 3
- net /USB_BOOT: track 4.65 -> 16.6 mm
- net -BATT: track 151.3 -> 158.9 mm, vias 22 -> 27
- net /MIC_DOUT_2: track 22.1 -> 18.6 mm
- net +3V3: track 115.9 -> 113.2 mm
- net Net-(D1-Pad2): track 2.13 -> 0.00 mm, vias 1 -> 0
- net /MIC_DOUT_1: track 20.2 -> 18.2 mm
- net Net-(D1-Pad1): track 0.00 -> 1.72 mm, vias 0 -> 1
- net /MIC_DOUT_0: track 22.4 -> 21.2 mm
- net +VDC: track 26.1 -> 27.0 mm
- net /MIC_DOUT_3: track 21.2 -> 22.0 mm
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Other:
- outline, holes or cut-outs redrawn
- board text added: "+"
- board text added: "-"
- board text added: "MSA Glasses v0.2 Design: Cayden Pierce"
