File: electronics_and_firmware/endpiece_mic_board_v0p1/microphone.kicad_pcb (KiCad board)
At the start: 2 copper layers, 5.1 x 5.8 mm, 7 parts, among them J1 PDM Mic, U1 MIC

Commit message: add gerbers for endpiece board
Parts:
- turned G1 to 180 degrees
Changed lines of the file:
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@@
       (layerselection 0x00010fc_ffffffff)
       (disableapertmacros false)
-      (usegerberextensions false)
-      (usegerberattributes false)
+      (usegerberextensions true)
+      (usegerberattributes true)
       (usegerberadvancedattributes false)
       (creategerberjobfile false)
@@
       (psa4output false)
       (plotreference true)
-      (plotvalue true)
+      (plotvalue false)
       (plotinvisibletext false)
       (sketchpadsonfab false)
-      (subtractmaskfromsilk false)
+      (subtractmaskfromsilk true)
       (outputformat 1)
       (mirror false)
-      (drillshape 1)
+      (drillshape 0)
       (scaleselection 1)
-      (outputdirectory "")
+      (outputdirectory "gerbers/")
     )
   )
@@
   (net 5 "Net-(J1-Pad3)")
   (footprint "Pauls_KiCAD_Libraries:Microhone_Graphic_sml" (layer "F.Cu")
-    (at 150.876 96.1009)
+    (at 150.876 96.1009 180)
     (property "Sheetfile" "/home/cayden/devdir/OpenSourceSmartGlasses/electronics_and_software/pcb/endpiece_mic_board_v0p1/microphone.sch")
     (property "Sheetname" "")
