File: electronics_and_firmware/OSSG_v0p4/OSSG_v0p4.kicad_pcb (KiCad board)
At the start: 4 copper layers, 85 x 9 mm, 71 parts, among them IC1 DW01A, J1 USB_B_Micro, J2 External PDM Mic Input, Q1 FS8205A, Q2 Q_NPN_BEC, Q3 Q_NPN_BEC, Q4 Q_PMOS_GSD, SW1 SW_SPST, U1 ESP32-PICO-D4, U2 TP4056, U3 NCP167BMX330TBG, U4 CH9102F, U5 XC61CC3002MR, U6 MP23DB01HPTR

Commit message: V0.4.1 schematic
Parts:
- removed IC1: DW01A, Package_TO_SOT_SMD:SOT-23-6
- removed TP18: GND_BO, OSSG_footprints:Breakout_pads
- removed TP19: IO21_BO, OSSG_footprints:Breakout_pads_small
- removed TP20: IO14_BO, OSSG_footprints:Breakout_pads_small
- removed TP21: IO5_BO, OSSG_footprints:Breakout_pads_small
- removed TP22: IO32_BO, OSSG_footprints:Breakout_pads_small
- removed TP24: IO33_BO, OSSG_footprints:Breakout_pads_small
- added C13: 1uF/16V, Capacitor_SMD:C_0402_1005Metric, F.Cu at (130.6, 100.9)
- added C14: 1uF/16V, Capacitor_SMD:C_0402_1005Metric, F.Cu at (122.9, 106.3)
- added C19: 1uF, Capacitor_SMD:C_0402_1005Metric, F.Cu at (127.7, 102.8)
- added D3: WS2812C-2020, OSSG_footprints:LED_WS2812C-2020, F.Cu at (145.5, 97.0)
- added D4: WS2812C-2020, OSSG_footprints:LED_WS2812C-2020, F.Cu at (141.0, 97.0)
- added D6: LED, Diode_SMD:D_0402_1005Metric, F.Cu at (120.3, 104.3)
- added D7: RB160M-30, Diode_SMD:D_SOD-123, F.Cu at (115.7, 105.0)
- added JP1: SolderJumper_2_Open, OSSG_footprints:JUMPER-2Psml_Open_RoundedPad2x1mm, F.Cu at (124.6, 101.4)
- added R17: .025, Resistor_SMD:R_0402_1005Metric, F.Cu at (127.8, 100.9)
- added R18: 100K, Resistor_SMD:R_0402_1005Metric, F.Cu at (123.2, 104.3)
- added R19: 884K, Resistor_SMD:R_0402_1005Metric, F.Cu at (132.5, 98.8)
- added R20: 100K, Resistor_SMD:R_0402_1005Metric, F.Cu at (120.0, 106.3)
- added R3: 10K, Resistor_SMD:R_0402_1005Metric, F.Cu at (149.0, 96.2)
- added SW2: Power, OSSG_footprints:SW_SMD_SPDT_Slide_9x6.9-hole, F.Cu at (113.6, 97.8)
- added TH1: 10K, Connector_PinHeader_1.27mm:PinHeader_1x02_P1.27mm_Horizontal, F.Cu at (124.5, 96.9)
- added TP12: IO0_TP, TestPoint:TestPoint_Pad_D1.0mm, F.Cu at (143.1, 100.3)
- added TP5: EN_TP, TestPoint:TestPoint_Pad_D1.0mm, F.Cu at (140.1, 100.3)
- added U7: NCP167BMX330TBG, OSSG_footprints:REG_NCP167BMX330TBG, F.Cu at (132.8, 96.5)
- C1: value 1uF -> 100nF
- C10, C11, C7, C8: value 1uF -> 0.1uF
- C15: value 100nF/C0G -> 100nF/16V
- C16: value 1uF/C0G -> 22uF/16V
- C17, C20, C9: value 0.1uF -> 1uF
- C18, C4: value 0.1uF -> 10uF
- C2: value 10uF -> 1uF
- C3: value 0.1uF -> 200pF
- D1, D2: value LED -> WS2812C-2020; footprint Diode_SMD:D_0402_1005Metric -> OSSG_footprints:LED_WS2812C-2020
- D5: value RB160M-30 -> LED; footprint Diode_SMD:D_SOD-123 -> Diode_SMD:D_0402_1005Metric
- J1: value USB_B_Micro -> Conn_01x05_Male; footprint Connector_USB:USB_Micro-B_Amphenol_10118194_Horizontal -> Connector_PinHeader_1.00mm:PinHeader_1x05_P1.00mm_Horizontal
- J2: value External PDM Mic Input -> USB_B_Micro; footprint OSSG_footprints:Solder-4P-Connector -> Connector_USB:USB_Micro-B_Amphenol_10118194_Horizontal
- Q1: value FS8205A -> 2SC4617R BR; footprint Package_TO_SOT_SMD:SOT-23-6 -> Package_TO_SOT_SMD:SOT-523
- Q2: value Q_NPN_BEC -> 2SC4617R BR
- Q3: value Q_NPN_BEC -> PMZ290UNE2YL; footprint Package_TO_SOT_SMD:SOT-523 -> OSSG_footprints:DFN100X60X40-3N
- Q4: value Q_PMOS_GSD -> EMF20B02V; footprint Package_TO_SOT_SMD:SOT-883 -> Package_TO_SOT_SMD:SOT-23-6
- R1: value 100 -> 0R*
- R10: value 100k -> 100K
- R11: value NC -> 442K; footprint Resistor_SMD:R_0201_0603Metric -> Resistor_SMD:R_0402_1005Metric
- R14: value 10K -> 160K
- R15: value 10K -> 884K
- R16: value 100k -> 320K
- R2: value 10K -> 0R*
- R4: value 1K -> 10K
- R5: value 4K -> 10K
- R6: value 10K* -> 100k
- R7: value 10K* -> 10K
- R8, R9: value 1k -> 2K
- TP1: value IO4_BO -> IO25_BO
- TP10: value IO37_ADC1C0 -> IO5_BO
- TP11: value IO38_ADC1C1 -> IO18_BO
- TP13: value +LBatt -> TXIN; footprint OSSG_footprints:Breakout_pads -> TestPoint:TestPoint_Pad_D1.0mm
- TP14: value -LBatt -> RXIN; footprint OSSG_footprints:Breakout_pads -> TestPoint:TestPoint_Pad_D1.0mm
- TP15: value +RBatt -> Batt+
- TP16: value -RBatt -> GND
- TP17: value +3.3V_BO -> BattMid
- TP2: value IO18_BO -> IO26_BO
- TP3: value TXIN -> IO38_ADC1C1; footprint TestPoint:TestPoint_Pad_D1.0mm -> OSSG_footprints:Breakout_pads_small
- TP4: value RXIN -> IO37_ADC1C0; footprint TestPoint:TestPoint_Pad_D1.0mm -> OSSG_footprints:Breakout_pads_small
- TP6: value IO25_BO -> IO32_BO
- TP7: value IO26_BO -> IO33_BO
- TP8: value EN_TP -> +3.3V_BO; footprint TestPoint:TestPoint_Pad_D1.0mm -> OSSG_footprints:Breakout_pads
- TP9: value IO0_TP -> GND_BO; footprint TestPoint:TestPoint_Pad_D1.0mm -> OSSG_footprints:Breakout_pads
- U1: value ESP32-PICO-D4 -> SPH0645LMH; footprint OSSG_footprints:ESP32_PICO_D4 -> OSSG_footprints:SPH0645LM4H-B-SMD-GND
- U2: value TP4056 -> ESP32-PICO-D4; footprint Package_SO:SOP-8_5.28x5.23mm_P1.27mm -> OSSG_footprints:ESP32_PICO_D4
- U3: value NCP167BMX330TBG -> CH9102F; footprint OSSG_footprints:REG_NCP167BMX330TBG -> Package_DFN_QFN:QFN-24-1EP_4x4mm_P0.5mm_EP2.6x2.6mm
- U4: value CH9102F -> XC61CC3002MR; footprint Package_DFN_QFN:QFN-24-1EP_4x4mm_P0.5mm_EP2.6x2.6mm -> Package_TO_SOT_SMD:SOT-23
- U5: value XC61CC3002MR -> MP2615CGQ-Z; footprint Package_TO_SOT_SMD:SOT-23 -> OSSG_footprints:MP2615GQ-P
- U6: value MP23DB01HPTR -> H7650-50PR; footprint OSSG_footprints:MP23DB01HPTR -> Package_TO_SOT_SMD:SOT-89-3
Connections:
- C1 pad 1: EN -> +3V3
- C1 pad 2: GND -> BATT2-
- C10 pad 1: GND -> Net-(C10-Pad1)
- C10 pad 2: V_PSU -> BATT2-
- C11 pad 1: GND -> +3V3
- C11 pad 2: +3V3 -> BATT2-
- C12 pad 1: Net-(C12-Pad1) -> BATT1-
- C12 pad 2: BATT- -> BATT2-
- C15 pad 1: GND -> Net-(C15-Pad1)
- C15 pad 2: +3V3 -> Net-(C15-Pad2)
- C16 pad 1: GND -> BATT+
- C16 pad 2: +3V3 -> BATT2-
- C17 pad 1: BATT+ -> V_PSU
- C17 pad 2: GND -> BATT2-
- C18 pad 1: +3V3 -> +5V
- C18 pad 2: GND -> BATT2-
- C2 pad 1: +3.3VA -> EN
- C2 pad 2: GND -> BATT2-
- C20 pad 1: V_USB -> BATT2-
- C20 pad 2: GND -> +3V3
- C3 pad 1: ADC1C0 -> BATT2-
- C3 pad 2: GND -> +3V3
- C4 pad 1: ADC1C1 -> Net-(C4-Pad1)
- C4 pad 2: GND -> BATT2-
- C5 pad 1: +3.3VA -> Net-(C4-Pad1)
- C5 pad 2: GND -> BATT2-
- C6 pad 1: ADC1C2 -> ADC1C0
- C6 pad 2: GND -> BATT2-
- C7 pad 1: GND -> ADC1C1
- C7 pad 2: V_PSU -> BATT2-
- C8 pad 1: GND -> ADC1C2
- C8 pad 2: V_USB -> BATT2-
- C9 pad 1: Net-(C9-Pad1) -> BATT2-
- C9 pad 2: GND -> V_USB
- D1 pad 2: Net-(D1-Pad2) -> BATT2-
- D2 pad 2: Net-(D2-Pad2) -> BATT2-
- D5 pad 1: V_PSU -> Net-(D5-Pad1)
- J1 pad 1: V_USB -> +3V3
- J1 pad 2: USB- -> BATT2-
- J1 pad 3: USB+ -> IO21
- J1 pad 4: unconnected-(J1-Pad4) -> IO23
- J1 pad 5: GND -> IO9
- J2 pad 1: +3V3 -> V_USB
- J2 pad 2: GND -> USB-
- J2 pad 3: EXT1_MIC_CLK -> USB+
- J2 pad 4: EXT1_MIC_DATA -> unconnected-(J2-Pad4)
- Q1 pad 1: GND -> Net-(Q1-Pad1)
- Q1 pad 2: unconnected-(Q1-Pad2) -> RTS
- Q1 pad 3: BATT- -> EN
- Q2 pad 2: RTS -> DTR
- Q2 pad 3: EN -> IO0
- Q3 pad 1: Net-(Q3-Pad1) -> PSEN
- Q3 pad 2: DTR -> BATT2-
- Q3 pad 3: IO0 -> Net-(Q3-Pad3)
- Q4 pad 1: V_USB -> BATT+
- Q4 pad 2: V_PSU -> Net-(Q3-Pad3)
- Q4 pad 3: BATT+ -> V_PSU
- R1 pad 1: BATT+ -> Net-(R1-Pad1)
- R1 pad 2: Net-(C12-Pad1) -> +3V3
- R10 pad 1: BATT+ -> BATT2-
- R10 pad 2: PSEN -> Net-(R10-Pad2)
- R11 pad 1: PSEN -> BATT+
- R11 pad 2: V_PSU -> Net-(R11-Pad2)
- R12 pad 1: BATT+ -> Net-(R11-Pad2)
- R13 pad 2: GND -> Net-(R13-Pad2)
- R14 pad 1: DTR -> Net-(R13-Pad2)
- R14 pad 2: Net-(Q2-Pad1) -> BATT2-
- R15 pad 1: RTS -> BATT+
- R15 pad 2: Net-(Q3-Pad1) -> ADC1C2
- R16 pad 1: GND -> ADC1C2
- R16 pad 2: V_USB -> BATT2-
- R2 pad 1: EN -> BATT2-
- R2 pad 2: +3V3 -> Net-(R1-Pad1)
- R4 pad 1: Net-(IC1-Pad2) -> DTR
- R4 pad 2: GND -> Net-(Q1-Pad1)
- R5 pad 1: GND -> RTS
- R5 pad 2: Net-(R5-Pad2) -> Net-(Q2-Pad1)
- R6 pad 1: Net-(R6-Pad1) -> BATT1-
- R6 pad 2: +3V3 -> PSEN
- R7 pad 1: GND -> Net-(C13-Pad1)
- R7 pad 2: Net-(R6-Pad1) -> Net-(R7-Pad2)
- R8 pad 1: V_USB -> Net-(D6-Pad1)
- R8 pad 2: Net-(D1-Pad2) -> Net-(R8-Pad2)
- R9 pad 1: V_USB -> Net-(D5-Pad1)
- R9 pad 2: Net-(D2-Pad2) -> Net-(R9-Pad2)
- SW1 pad 1: GND -> BATT2-
- TP1 pad 1: IO4 -> IO25
- TP10 pad 1: ADC1C0 -> IO5
- TP11 pad 1: ADC1C1 -> IO18
- TP13 pad 1: BATT+ -> TX_ESP
- TP14 pad 1: BATT- -> RX_ESP
- TP16 pad 1: BATT- -> BATT2-
- TP17 pad 1: +3V3 -> BATT1-
- TP2 pad 1: IO18 -> IO26
- TP3 pad 1: TX_ESP -> ADC1C1
- TP4 pad 1: RX_ESP -> ADC1C0
- TP6 pad 1: IO25 -> IO32
- TP7 pad 1: IO26 -> IO33
- TP8 pad 1: EN -> +3V3
- TP9 pad 1: IO0 -> BATT2-
- U1 pad 1: +3.3VA -> IO33
- U1 pad 2: Net-(AE1-Pad2) -> Net-(R1-Pad1)
- U1 pad 3: +3.3VA -> BATT2-
- U1 pad 4: +3.3VA -> IO32
- U1 pad 5: ADC1C2 -> +3V3
- U1 pad 6: ADC1C0 -> IO14
- U2 pad 1: GND -> +3V3
- U2 pad 2: Net-(R5-Pad2) -> Net-(AE1-Pad2)
- U2 pad 3: GND -> +3V3
- U2 pad 4: V_USB -> +3V3
- U2 pad 5: BATT+ -> ADC1C2
- U2 pad 6: Net-(D1-Pad1) -> ADC1C0
- U2 pad 7: Net-(D2-Pad1) -> ADC1C1
- U2 pad 8: V_USB -> IO39
- U3 pad 1: +3V3 -> unconnected-(U3-Pad1)
- U3 pad 2: GND -> BATT2-
- U3 pad 3: PSEN -> USB+
- U3 pad 4: V_PSU -> USB-
- U3 pad 5: GND -> +3V3
- U4 pad 1: unconnected-(U4-Pad1) -> PSEN
- U4 pad 2: GND -> BATT2-
- U4 pad 3: USB+ -> BATT1-
- U5 pad 1: PSEN -> Net-(C15-Pad2)
- U5 pad 2: GND -> V_USB
- U5 pad 3: BATT+ -> Net-(R7-Pad2)
- U6 pad 1: IO32 -> BATT2-
- U6 pad 2: Net-(R6-Pad1) -> V_PSU
- U6 pad 3: GND -> +5V
Routing:
- net BATT2-: track 0.00 -> 442.0 mm, vias 0 -> 73
- net GND: track 51.3 -> 0.35 mm, vias 56 -> 0
- net BATT+: track 47.3 -> 0.00 mm, vias 4 -> 0
- net V_USB: track 46.4 -> 0.00 mm, vias 2 -> 0
- net ADC1C2: track 41.5 -> 5.17 mm, vias 3 -> 2
- net +3V3: track 27.9 -> 3.19 mm, vias 9 -> 2
- net IO32: track 31.4 -> 11.8 mm, vias 2 -> 3
- net EN: track 34.5 -> 15.0 mm, vias 3 -> 2
- net PSEN: track 19.4 -> 0.00 mm, vias 3 -> 0
- net BATT-: track 17.4 -> 0.00 mm, vias 1 -> 0
- net IO33: track 32.1 -> 15.9 mm, vias 1 -> 2
- net +3.3VA: track 15.0 -> 0.00 mm, vias 3 -> 0
- net V_PSU: track 13.3 -> 0.00 mm, vias 3 -> 0
- net IO26: track 15.9 -> 3.01 mm, vias 2 -> 1
- net TX_ESP: track 12.6 -> 0.00 mm, vias 1 -> 0
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- added copper zone on B.Cu, net +5V
- added copper zone on F.Cu, net +5V
- added copper zone on In1.Cu, net +5V
- added copper zone on In2.Cu, net +5V
- added copper zone on B.Cu, net BATT2-
- added copper zone on F.Cu, net BATT2-
- added copper zone on In1.Cu, net BATT2-
- removed copper zone on B.Cu, net GND
- removed copper zone on F.Cu, net GND
- removed copper zone on In1.Cu, net GND
- removed copper zone on In2.Cu, net GND
