File: electronics_and_firmware/OSSG_v0p4-2P/Power.kicad_sch (KiCad schematic)
At the start: 38 parts, among them J2 USB_B_Micro, Q3 PMZ290UNE2YL, Q4 EMF20B02V, SW2 Power, U4 XC61CC3002MR, U5 MP2615CGQ-Z, U6 H7650-50PR, U7 NCP167BMX330TBG

Commit message: finished beta 2 of V0.4-2P schematic
Parts:
- removed C14: 1uF/16V, Capacitor_SMD:C_0402_1005Metric, symbol Device:C_Small
- removed C15: 100nF/16V, Capacitor_SMD:C_0402_1005Metric, symbol Device:C_Small
- removed C17: 1uF, Capacitor_SMD:C_0402_1005Metric, symbol Device:C_Small
- removed D5, D6: LED, Diode_SMD:D_0402_1005Metric, symbol Device:LED
- removed JP1: SolderJumper_2_Open, OSSG_footprints:JUMPER-2Psml_Open_RoundedPad2x1mm, symbol Jumper:SolderJumper_2_Open
- removed R10, R9: 2K, Resistor_SMD:R_0402_1005Metric, symbol Device:R
- removed R11: 100K, Resistor_SMD:R_0402_1005Metric, symbol Device:R
- removed R14: .025, Resistor_SMD:R_0402_1005Metric, symbol Device:R
- removed R8: 10K, Resistor_SMD:R_0402_1005Metric, symbol Device:R
- removed TH1: 10K, Connector_PinHeader_1.27mm:PinHeader_1x02_P1.27mm_Horizontal, symbol Device:Thermistor_NTC
- removed U5: MP2615CGQ-Z, OSSG_footprints:MP2615GQ-P, symbol OSSG_components_lib:MP2615CGQ-Z
- removed U6: H7650-50PR, Package_TO_SOT_SMD:SOT-89-3, symbol OSSG_components_lib:H7650
- added C16: 1uF, Capacitor_SMD:C_0402_1005Metric, symbol Device:C_Small
- added C18, C20: 22uF, Capacitor_SMD:C_0402_1005Metric, symbol Device:C_Small
- added D5: Red, Diode_SMD:D_0402_1005Metric, symbol Device:LED_Small
- added R7: 2K, Resistor_SMD:R_0402_1005Metric, symbol Device:R_Small
- added U5: AP5054HTC, Package_TO_SOT_SMD:SOT-23-6, symbol OSSG_components_lib:AP5054HTC
- added U6: MAX17048, Package_DFN_QFN:DFN-8-1EP_2x2mm_P0.5mm_EP0.8x1.6mm, symbol OSSG_components_lib:MAX17048
- added U8: SY7088, Package_DFN_QFN:DFN-8-1EP_3x2mm_P0.5mm_EP1.7x1.4mm, symbol OSSG_components_lib:SY7088
- C13: value 1uF/16V -> 100nF
- C17: renamed from C18; value 10uF -> 100nF
- L1: value 6.8uH -> 1.5uH; footprint (none) -> OSSG_footprints:1.5uH_YXMAA0402-1R5M-ANP; P/N (none) -> C241335
- R12: value 884K -> 470K; MPN_LCSC C106234 -> 1
- R13: value 320K -> 147K; MPN_LCSC C106234 -> 1
- TP17: value BattMid -> 5V
- renumbered C16 to C14, C19 to C15, C20 to C19, D7 to D6, R16 to R10, R17 to R11, R7 to R8, R15 to R9
Connections:
- net V_PSU is gone; now on an unnamed net: C15.2, D6.1 (K), Q4.3 (S2)
- net V_USB is gone; now on net VBUS: D6.2 (A), Q4.4 (G2), R11.2
- net +5V: now also R12.2, TP17.1, C20.1, U8.7 (OUT), U8.8 (OUT)
- net BATT+: now also C12.1, C13.1, R6.1, U4.3 (VIN), U5.3 (BAT), U6.2 (CELL), U6.3 (Vdd); no longer R12.1
- net GND: now also R13.1, C16.2, C18.2, C20.2, R7.1, U5.2 (GND), U6.1 (CTG), U6.4 (GND), U6.6 (QSTRT), U6.9 (EP), U8.4 (GND), U8.9 (Pad); no longer R13.2
- net PSEN: now also R6.2, R8.1, U4.1 (VOUT), U8.3 (EN); no longer Q3.1 (G), R8.2, R9.2
- net at L1.1: now also C16.1, C18.1, U8.6 (IN)
- net at L1.2: now also U8.1 (LX), U8.2 (LX)
- net VBUS: now reaches J2.1 (VBUS)
- net VBUS: now also D5.2 (A), U5.4 (VCC)
- removed net BATT1-: C12.1, R6.1, TP17.1, U4.3 (VIN)
- removed net IO36: R12.2, R13.1
- new net: R12.1, R13.2, U8.5 (FB)
- new net: Q3.1 (G), R8.2, R9.2
- new net: D5.1 (K), U5.1 (~{CHRG})
- new net: R7.2, U5.6 (PROG)
- new net ALRT: U6.5 (ALRT)
- new net SCL: U6.7 (SCL)
- new net SDA: U6.8 (SDA)
Other:
- note added: "2.7V-4.2V"
- note added: "2.7V-4.7V"
- note added: "2.7V-4.7V to 5V Boost"
- note added: "2K=500mA charge"
- note added: "500mA LiPo Battery Charger"
- note added: "5V to 3.3V LDO"
- note added: "Battery Bypass"
- note added: "Battery Fuel Gauge"
- note added: "Dual LiPo 2.7V to 4.2V 500mA Batteries"
- note added: "Power On/Off + Low Battery Isolation"
- note added: "USB In"
- note added: "will be supplying 22mA to GND while switched on"
- note removed: "* Note: need to test how well the H7650 LDO passes the USB 4.6V thru to the otherside"
- note removed: "10V to 5V LDO Up to 750mA"
- note removed: "1589-MP2615CGQ-ZCT-ND Digikey P/N - A$3.66/ea 946-MP2615GQ-Z Mouser P/N - US$2.37/ea"
- note removed: "4.6V - 8.2V"
- note removed: "5V to 12V at 1.5A Boost DC-Dc converter"
- note removed: "6V-8.4V"
- note removed: "Battery Voltage Sense"
- note removed: "Lipo charging and protection"
- note removed: "Power Supply Regulator"
- note removed: "Power Supply Switching"
- note removed: "SELL float for 4.2V battery or to GND for 4.1V battery"
- note removed: "SY7088 IC"
- note removed: "USB"
- note removed: "ind. DC Res below 50m ohms"
- note removed: "leave CELL floating for 2S Battery"
- note removed: "will be supplying 50mA to GND while switched on"
- moved on the sheet: C12, C14, C15, D6, J2, Q3, Q4A, Q4B, R10, R11, R6, R8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

Commit message: started work on PCB layout
Parts:
- removed C15: 1uF, Capacitor_SMD:C_0402_1005Metric, symbol Device:C_Small
- added TP15: Batt1+, OSSG_footprints:Breakout_pads, symbol Connector:TestPoint
- added TP17: BATT1-, OSSG_footprints:Breakout_pads, symbol Connector:TestPoint
- Q4: footprint Package_TO_SOT_SMD:SOT-23-6 -> OSSG_footprints:EMF20B02V
- R10: value 884K -> 1M
- R11: value 100K -> 1M
- SW2: P/N (none) -> C145858
- TP16: renamed from TP15; value Batt+ -> Batt2+
- TP18: renamed from TP16; value GND -> BATT2-
- TP19: renamed from TP17; footprint OSSG_footprints:Breakout_pads -> OSSG_footprints:Breakout_pads_small
- renumbered C16 to C15, C17 to C16, C18 to C17, C19 to C18, C20 to C19
Connections:
- net BATT+: now also TP15.1
- net GND: now also TP17.1
Other:
- moved on the sheet: TP16

Commit message: V0.4-2P PCB nearly finished
Parts:
- added F1: 1A, Resistor_SMD:R_0805_2012Metric, symbol Device:Polyfuse_Small
- renumbered D5 to D2, D6 to D3, J2 to J3, R9 to R10, R10 to R11, R11 to R12, R12 to R13, R13 to R14, R6 to R7, R7 to R8, R8 to R9
Connections:
- net VBUS: now also F1.2; no longer J3.1 (VBUS)
- net at Q4.5 (D2), Q4.7 (D2): now also Q4.6 (D2), Q4.8 (D2)
- new net: F1.1, J3.1 (VBUS)
